File: KNXBusankoppler.sch (KiCad schematic (older format))
At the start: 3 parts, among them J1 Conn_01x10_Male, J2 Conn_01x04_Male, U1 ProMicro

Commit message: CO2-Sensor 1.0
Parts:
- added C1: 25v 2200uf, Capacitor_THT:CP_Radial_D10.0mm_P5.00mm_P7.50mm, symbol Device:CP
- added C2: 6.3v 1000uf, Capacitor_THT:CP_Radial_D8.0mm_P3.80mm, symbol Device:CP
- added D1, D2, D3: LED, LED_SMD:LED_0805_2012Metric_Pad1.15x1.40mm_HandSolder, symbol Device:LED
- added J3: Screw_Terminal_01x02, TerminalBlock:TerminalBlock_bornier-2_P5.08mm, symbol Connector:Screw_Terminal_01x02
- added R1, R2, R3: R, Resistor_SMD:R_0805_2012Metric_Pad1.15x1.40mm_HandSolder, symbol Device:R
- added SW1: SW_Push, Button_Switch_SMD:SW_SPST_CK_RS282G05A3, symbol Switch:SW_Push
- added U2: MH_Z19B, libs:MH-Z19B, symbol haus-automatisierung:MH_Z19B
- added U3: MP1584, libs:MP1584_buck_module_SMD, symbol KNXBusankoppler-rescue:MP1584-haus-automatisierung
- U1: footprint libs:ProMicro -> libs:ProMicroSMD
Connections:
- net GND: now also U1.23 (GND), C1.2, C2.2, D1.1 (K), D2.1 (K), D3.1 (K), J3.2 (Pin_2), SW1.2, U2.2 (GND), U3.2 (In-), U3.4 (Out-)
- net 20V: now reaches J1.6 (Pin_6)
- net 20V: now also C1.1, U3.1 (In+)
- net at U1.11 (B4): now also U2.7 (Tx)
- net at U1.12 (B5): now also U2.6 (Rx)
- net at U1.13 (B6): now also R3.2
- net at U1.14 (B2): now also R2.2
- net at U1.15 (B3): now also R1.2
- net at U1.16 (B1): now also J3.1 (Pin_1), SW1.1
- new net: C2.1, U2.1 (Vin), U3.3 (Out+)
- new net: D1.2 (A), R1.1
- new net: D2.2 (A), R2.1
- new net: D3.2 (A), R3.1
- no-connect marks 6 -> 21

Commit message: Changed Footprint
Parts:
- U1: footprint libs:ProMicroSMD -> halibs:ArduinoProMicroSMD
- U2: footprint libs:MH-Z19B -> halibs:MH-Z19B
Changed lines of the file:
@@
 Sheet 1 1
 Title "KNX-Busankoppler"
-Date "2019-04-17"
+Date "2019-05-11"
 Rev "1.1"
 Comp "haus-automatisierung.com"
@@
 NoConn ~ 3100 3450
 NoConn ~ 3100 3950
-$Comp
-L promicro:ProMicro U1
-U 1 1 5CB6F800
-P 6100 3600
-F 0 "U1" H 6100 4637 60  0000 C CNN
-F 1 "ProMicro" H 6100 4531 60  0000 C CNN
-F 2 "libs:ProMicroSMD" H 6200 2550 60  0001 C CNN
-F 3 "" H 6200 2550 60  0000 C CNN
-	1    6100 3600
-	1    0    0    -1
-$EndComp
 Wire Wire Line
 	3100 3050 3400 3050
@@
 F 0 "U2" H 6550 4850 50  0000 C CNN
 F 1 "MH_Z19B" H 6900 4850 50  0000 C CNN
-F 2 "libs:MH-Z19B" H 6700 5100 50  0001 C CNN
+F 2 "halibs:MH-Z19B" H 6700 5100 50  0001 C CNN
 F 3 "" H 6700 5100 50  0001 C CNN
 	1    6700 5100
@@
 	7900 3950 7900 3850
 Connection ~ 7900 3850
-Text Label 6900 2950 0    50   ~ 0
-GND
 Wire Wire Line
 	7100 3550 6950 3550
@@
 	1    0    0    -1
 $EndComp
+Wire Wire Line
+	7350 3400 7600 3400
+Wire Wire Line
+	7600 3400 7600 3550
+Wire Wire Line
+	7600 3550 7500 3550
+Wire Wire Line
+	7250 3400 6950 3400
+Wire Wire Line
+	6950 3400 6950 3550
+Connection ~ 6950 3550
+Text Label 5400 5700 0    50   ~ 0
+GND
+Wire Wire Line
+	7600 3550 7900 3550
+Connection ~ 7600 3550
+Connection ~ 7900 3550
+Wire Wire Line
+	7900 3550 7900 2950
+$Comp
+L promicro:ProMicro U1
+U 1 1 5CB6F800
+P 6100 3600
+F 0 "U1" H 6100 4637 60  0000 C CNN
+F 1 "ProMicro" H 6100 4531 60  0000 C CNN
+F 2 "halibs:ArduinoProMicroSMD" H 6200 2550 60  0001 C CNN
+F 3 "" H 6200 2550 60  0000 C CNN
+	1    6100 3600
+	1    0    0    -1
+$EndComp
+Text Label 6900 2950 0    50   ~ 0
+GND
 $Comp
 L Connector:Screw_Terminal_01x02 J3
@@
 	0    -1   -1   0
 $EndComp
-Wire Wire Line
-	7350 3400 7600 3400
-Wire Wire Line
-	7600 3400 7600 3550
-Wire Wire Line
-	7600 3550 7500 3550
-Wire Wire Line
-	7250 3400 6950 3400
-Wire Wire Line
-	6950 3400 6950 3550
-Connection ~ 6950 3550
-Text Label 5400 5700 0    50   ~ 0
-GND
 NoConn ~ 6800 3150
-Wire Wire Line
-	7600 3550 7900 3550
-Connection ~ 7600 3550
-Connection ~ 7900 3550
-Wire Wire Line
-	7900 3550 7900 2950
 $EndSCHEMATC
