File: KNXBusankoppler.sch (KiCad schematic (older format))
At the start: 3 parts, among them J1 Conn_01x10_Male, J2 Conn_01x04_Male, U1 ProMicro

Commit message: v1.1
Parts:
- U1: footprint libs:ProMicro -> halibs:ArduinoProMicro
Changed lines of the file:
@@
 EESchema Schematic File Version 4
 LIBS:KNXBusankoppler-cache
-EELAYER 26 0
+EELAYER 29 0
 EELAYER END
 $Descr A4 11693 8268
@@
 Sheet 1 1
 Title "KNX-Busankoppler"
-Date "2019-04-17"
-Rev "1.0"
+Date "2019-05-17"
+Rev "1.1"
 Comp "haus-automatisierung.com"
 Comment1 "Matthias Kleine"
@@
 F 0 "U1" H 6100 4637 60  0000 C CNN
 F 1 "ProMicro" H 6100 4531 60  0000 C CNN
-F 2 "libs:ProMicro" H 6200 2550 60  0001 C CNN
+F 2 "halibs:ArduinoProMicro" H 6200 2550 60  0001 C CNN
 F 3 "" H 6200 2550 60  0000 C CNN
 	1    6100 3600
@@
 RX
 $Comp
-L power:GND #PWR?
+L power:GND #PWR0101
 U 1 1 5CB71BCE
 P 3400 2850
-F 0 "#PWR?" H 3400 2600 50  0001 C CNN
+F 0 "#PWR0101" H 3400 2600 50  0001 C CNN
 F 1 "GND" H 3405 2677 50  0000 C CNN
 F 2 "" H 3400 2850 50  0001 C CNN
