File: KNXBusankoppler.kicad_pcb (KiCad board)
At the start: 2 copper layers, 42.2 x 37.3 mm, 6 parts, among them J1 Conn_01x10_Male, J2 Conn_01x04_Male, U1 ProMicro

Commit message: v1.1
Parts:
- U1: footprint libs:ProMicro -> halibs:ArduinoProMicro
- moved G*** 15.1 mm to (127.8, 91.1)
- moved U1 6.26 mm to (138.7, 91.1)
Routing:
- net GND: track 41.4 -> 0.00 mm
- net /RX: track 51.2 -> 45.0 mm
- net /TX: track 52.1 -> 49.1 mm
- net /5V: track 61.8 -> 59.7 mm
Other:
- board text added: "v1.1"
- board text removed: "v1.0"

Commit message: Updated to KiCad 6
Parts:
- U1: footprint halibs:ArduinoProMicro -> haus-automatisierung:ArduinoProMicro
Connections:
- J1 pad 10: Net-(J1-Pad10) -> unconnected-(J1-Pad10)
- J1 pad 2: Net-(J1-Pad2) -> unconnected-(J1-Pad2)
- J1 pad 4: Net-(J1-Pad4) -> unconnected-(J1-Pad4)
- J1 pad 5: Net-(J1-Pad5) -> unconnected-(J1-Pad5)
- J1 pad 6: Net-(J1-Pad6) -> unconnected-(J1-Pad6)
- J1 pad 8: Net-(J1-Pad8) -> unconnected-(J1-Pad8)
- U1 pad 10: Net-(U1-Pad10) -> unconnected-(U1-Pad10)
- U1 pad 11: Net-(U1-Pad11) -> unconnected-(U1-Pad11)
- U1 pad 12: Net-(U1-Pad12) -> unconnected-(U1-Pad12)
- U1 pad 13: Net-(U1-Pad13) -> unconnected-(U1-Pad13)
- U1 pad 14: Net-(U1-Pad14) -> unconnected-(U1-Pad14)
- U1 pad 15: Net-(U1-Pad15) -> unconnected-(U1-Pad15)
- U1 pad 16: Net-(U1-Pad16) -> unconnected-(U1-Pad16)
- U1 pad 17: Net-(U1-Pad17) -> unconnected-(U1-Pad17)
- U1 pad 18: Net-(U1-Pad18) -> unconnected-(U1-Pad18)
- U1 pad 19: Net-(U1-Pad19) -> unconnected-(U1-Pad19)
- U1 pad 20: Net-(U1-Pad20) -> unconnected-(U1-Pad20)
- U1 pad 21: Net-(U1-Pad21) -> unconnected-(U1-Pad21)
- U1 pad 22: Net-(U1-Pad22) -> unconnected-(U1-Pad22)
- U1 pad 23: Net-(U1-Pad23) -> unconnected-(U1-Pad23)
- U1 pad 4: Net-(U1-Pad4) -> unconnected-(U1-Pad4)
- U1 pad 5: Net-(U1-Pad5) -> unconnected-(U1-Pad5)
- U1 pad 6: Net-(U1-Pad6) -> unconnected-(U1-Pad6)
- U1 pad 7: Net-(U1-Pad7) -> unconnected-(U1-Pad7)
- U1 pad 8: Net-(U1-Pad8) -> unconnected-(U1-Pad8)
- U1 pad 9: Net-(U1-Pad9) -> unconnected-(U1-Pad9)
Other:
- net class Default removed

Commit message: Updated preview / year 2024
Parts:
- removed G***: LOGO, libs:Logo
